Commit message: added gazebo launch files

File: urdf/robot.urdf.xacro (robot description, xacro)
@@ -2,3 +2,4 @@
 <robot xmlns:xacro="http://www.ros.org/wiki/xacro"  name="robot">
     <xacro:include filename="robot_structure.xacro" />
+    <xacro:include filename="diffdrive.xacro" />
 </robot>

File: urdf/robot_structure.xacro (robot description, xacro)
@@ -37,13 +37,16 @@
             </geometry>
         </collision>
-        <xacro:inertial_box mass="0.5" x="0.15" y="0.15" z="0.3">
+        <xacro:inertial_box mass="0.8" x="0.15" y="0.15" z="0.3">
             <origin xyz="0.075 0 0.1" rpy="0 0 0"/>
         </xacro:inertial_box>
     </link>
+    <gazebo reference="chassis">
+        <material>Gazebo/Blue</material>
+    </gazebo>
     <!-- LEFT WHEEL LINK -->
     <joint name="left_wheel_joint" type="continuous">
         <parent link="base_link"/>
         <child link="left_wheel"/>
-        <origin xyz="-0.015 0.085 0" rpy="-${pi/2} 0 0" />
+        <origin xyz="0.065 0.085 0" rpy="-${pi/2} 0 0" />
         <axis xyz="0 0 1"/>
     </joint>
@@ -60,13 +63,16 @@
             </geometry>
         </collision>
-        <xacro:inertial_cylinder mass="0.1" length="0.02" radius="0.035">
+        <xacro:inertial_cylinder mass="0.05" length="0.02" radius="0.035">
             <origin xyz="0 0 0" rpy="0 0 0"/>
         </xacro:inertial_cylinder>
     </link>
+    <gazebo reference="left_wheel">
+        <material>Gazebo/White</material>
+    </gazebo>
     <!-- RIGHT WHEEL LINK -->
     <joint name="right_wheel_joint" type="continuous">
         <parent link="base_link"/>
         <child link="right_wheel"/>
-        <origin xyz="-0.015 -0.085 0" rpy="${pi/2} 0 0" />
+        <origin xyz="0.065 -0.085 0" rpy="${pi/2} 0 0" />
         <axis xyz="0 0 -1"/>
     </joint>
@@ -83,18 +89,21 @@
             </geometry>
         </collision>
-        <xacro:inertial_cylinder mass="0.1" length="0.02" radius="0.035">
+        <xacro:inertial_cylinder mass="0.05" length="0.02" radius="0.035">
             <origin xyz="0 0 0" rpy="0 0 0"/>
         </xacro:inertial_cylinder>
     </link>
+    <gazebo reference="right_wheel">
+        <material>Gazebo/White</material>
+    </gazebo>
     <!-- CASTER WHEEL LINK -->
     <joint name="caster_wheel_joint_cylinder" type="fixed">
         <parent link="chassis"/>
         <child link="caster_wheel_cylinder"/>
-        <origin xyz="0.12 0 0"/>
+        <origin xyz="0.02 0 0"/>
     </joint>
     <link name="caster_wheel_cylinder">
         <visual>
             <geometry>
-                <cylinder radius="0.01" length="0.04"/>
+                <cylinder radius="0.01" length="0.05"/>
             </geometry>
             <material name="black"/>
@@ -102,15 +111,18 @@
         <collision>
             <geometry>
-                <cylinder radius="0.01" length="0.04"/>
+                <cylinder radius="0.01" length="0.05"/>
             </geometry>
         </collision>
-        <xacro:inertial_cylinder mass="0.01" length="0.04" radius="0.01">
+        <xacro:inertial_cylinder mass="0.5" length="0.05" radius="0.01">
             <origin xyz="0 0 0" rpy="0 0 0"/>
         </xacro:inertial_cylinder>
     </link>
+    <gazebo reference="caster_wheel_cylinder">
+        <material>Gazebo/Black</material>
+    </gazebo>
     <joint name="caster_wheel_joint_sphere" type="fixed">
         <parent link="chassis"/>
         <child link="caster_wheel_sphere"/>
-        <origin xyz="0.12 0 -0.02"/>
+        <origin xyz="0.02 0 -0.025"/>
     </joint>
     <link name="caster_wheel_sphere">
@@ -126,7 +138,12 @@
             </geometry>
         </collision>
-        <xacro:inertial_sphere mass="0.05" radius="0.01">
+        <xacro:inertial_sphere mass="0.5" radius="0.01">
             <origin xyz="0 0 0" rpy="0 0 0"/>
         </xacro:inertial_sphere>
     </link>
+    <gazebo reference="caster_wheel_sphere">
+        <material>Gazebo/White</material>
+        <mu1 value = "0.01"/>
+        <mu2 value = "0.01"/>
+    </gazebo>
 </robot>

Commit message: Multi robot spawning launch file created

File: urdf/robot.urdf.xacro (robot description, xacro)
@@ -3,3 +3,4 @@
     <xacro:include filename="robot_structure.xacro" />
     <xacro:include filename="diffdrive.xacro" />
+    <xacro:include filename="lidar.xacro" />
 </robot>

File: urdf/robot_structure.xacro (robot description, xacro)
@@ -37,5 +37,5 @@
             </geometry>
         </collision>
-        <xacro:inertial_box mass="0.8" x="0.15" y="0.15" z="0.3">
+        <xacro:inertial_box mass="1" x="0.15" y="0.15" z="0.3">
             <origin xyz="0.075 0 0.1" rpy="0 0 0"/>
         </xacro:inertial_box>
@@ -46,7 +46,7 @@
     <!-- LEFT WHEEL LINK -->
     <joint name="left_wheel_joint" type="continuous">
-        <parent link="base_link"/>
+        <parent link="chassis"/>
         <child link="left_wheel"/>
-        <origin xyz="0.065 0.085 0" rpy="-${pi/2} 0 0" />
+        <origin xyz="0.115 0.085 0" rpy="-${pi/2} 0 0" />
         <axis xyz="0 0 1"/>
     </joint>
@@ -72,7 +72,7 @@
     <!-- RIGHT WHEEL LINK -->
     <joint name="right_wheel_joint" type="continuous">
-        <parent link="base_link"/>
+        <parent link="chassis"/>
         <child link="right_wheel"/>
-        <origin xyz="0.065 -0.085 0" rpy="${pi/2} 0 0" />
+        <origin xyz="0.115 -0.085 0" rpy="${pi/2} 0 0" />
         <axis xyz="0 0 -1"/>
     </joint>
@@ -144,6 +144,6 @@
     <gazebo reference="caster_wheel_sphere">
         <material>Gazebo/White</material>
-        <mu1 value = "0.01"/>
-        <mu2 value = "0.01"/>
+        <mu1 value = "0.001"/>
+        <mu2 value = "0.001"/>
     </gazebo>
 </robot>
