Commit message: Resolved laser conflict

File: urdf/bot1.urdf.xacro (robot description, xacro)
@@ -123,8 +123,8 @@
     <joint name="/robot1/laser_joint" type="fixed">
         <parent link="/robot1/chassis"/>
-        <child link="/robot1/laser_frame"/>
+        <child link="laser_frame_1"/>
         <origin xyz="0.1 0 0.200" rpy="0 0 0"/>
     </joint>
-    <link name="/robot1/laser_frame">
+    <link name="laser_frame_1">
         <visual>
             <geometry>
@@ -142,5 +142,5 @@
         </xacro:inertial_cylinder>
     </link>
-    <gazebo reference="/robot1/laser_frame">
+    <gazebo reference="laser_frame_1">
         <material>Gazebo/Black</material>
         <sensor name="laser" type="ray">
@@ -166,5 +166,5 @@
                 </ros>
                 <output_type>sensor_msgs/LaserScan</output_type>
-                <frame_name>laser_frame_robot1</frame_name>
+                <frame_name>laser_frame_1</frame_name>
             </plugin>
         </sensor>

File: urdf/bot2.urdf.xacro (robot description, xacro)
@@ -123,8 +123,8 @@
     <joint name="/robot2/laser_joint" type="fixed">
         <parent link="/robot2/chassis"/>
-        <child link="/robot2/laser_frame"/>
+        <child link="laser_frame_2"/>
         <origin xyz="0.1 0 0.200" rpy="0 0 0"/>
     </joint>
-    <link name="/robot2/laser_frame">
+    <link name="laser_frame_2">
         <visual>
             <geometry>
@@ -142,5 +142,5 @@
         </xacro:inertial_cylinder>
     </link>
-    <gazebo reference="/robot2/laser_frame">
+    <gazebo reference="laser_frame_2">
         <material>Gazebo/Black</material>
         <sensor name="laser" type="ray">
@@ -166,5 +166,5 @@
                 </ros>
                 <output_type>sensor_msgs/LaserScan</output_type>
-                <frame_name>laser_frame_robot2</frame_name>
+                <frame_name>laser_frame_2</frame_name>
             </plugin>
         </sensor>
